Commit message: feat: make agx_arm_urdf a standalone ROS 2 package
- add ament_cmake package metadata
- add a prefix-aware Piper Xacro macro
- update mesh URIs to resolve from agx_arm_urdf
- document standalone and vcstool-based usage

File: nero/urdf/nero_description.urdf (robot description, URDF)
Before this commit: robot nero, 9 links, 8 joints
Links:
- link base_link: geometry collision mesh filename=package://agx_arm_urdf/nero/meshes/base_link.stl; visual mesh filename=package://agx_arm_urdf/nero/meshes/dae/base_link.dae
- link link1: geometry collision mesh filename=package://agx_arm_urdf/nero/meshes/link1.stl; visual mesh filename=package://agx_arm_urdf/nero/meshes/dae/link1.dae
- link link2: geometry collision mesh filename=package://agx_arm_urdf/nero/meshes/link2.stl; visual mesh filename=package://agx_arm_urdf/nero/meshes/dae/link2.dae
- link link3: geometry collision mesh filename=package://agx_arm_urdf/nero/meshes/link3.stl; visual mesh filename=package://agx_arm_urdf/nero/meshes/dae/link3.dae
- link link4: geometry collision mesh filename=package://agx_arm_urdf/nero/meshes/link4.stl; visual mesh filename=package://agx_arm_urdf/nero/meshes/dae/link4.dae
- link link5: geometry collision mesh filename=package://agx_arm_urdf/nero/meshes/link5.stl; visual mesh filename=package://agx_arm_urdf/nero/meshes/dae/link5.dae
- link link6: geometry collision mesh filename=package://agx_arm_urdf/nero/meshes/link6.stl; visual mesh filename=package://agx_arm_urdf/nero/meshes/dae/link6.dae
- link link7: geometry collision mesh filename=package://agx_arm_urdf/nero/meshes/link7.stl; visual mesh filename=package://agx_arm_urdf/nero/meshes/dae/link7.dae

File: nero/urdf/nero_with_gripper_description.xacro (robot description, xacro)
@@ -13,5 +13,5 @@
             <origin xyz="0 0 0" rpy="0 0 0"/>
             <geometry>
-                <mesh filename="package://agx_arm_description/agx_arm_urdf/nero/meshes/dae/gripper_base.dae"/>
+                <mesh filename="package://agx_arm_urdf/nero/meshes/dae/gripper_base.dae"/>
             </geometry>
         </visual>
@@ -19,5 +19,5 @@
             <origin xyz="0 0 0" rpy="0 0 0"/>
             <geometry>
-                <mesh filename="package://agx_arm_description/agx_arm_urdf/nero/meshes/gripper_base.stl"/>
+                <mesh filename="package://agx_arm_urdf/nero/meshes/gripper_base.stl"/>
             </geometry>
         </collision>
@@ -45,5 +45,5 @@
             <origin xyz="0 0 0" rpy="0 0 0"/>
             <geometry>
-                <mesh filename="package://agx_arm_description/agx_arm_urdf/nero/meshes/dae/gripper_link1.dae"/>
+                <mesh filename="package://agx_arm_urdf/nero/meshes/dae/gripper_link1.dae"/>
             </geometry>
         </visual>
@@ -51,5 +51,5 @@
             <origin xyz="0 0 0" rpy="0 0 0"/>
             <geometry>
-                <mesh filename="package://agx_arm_description/agx_arm_urdf/nero/meshes/gripper_link1.stl"/>
+                <mesh filename="package://agx_arm_urdf/nero/meshes/gripper_link1.stl"/>
             </geometry>
         </collision>
@@ -72,5 +72,5 @@
             <origin xyz="0 0 0" rpy="0 0 0"/>
             <geometry>
-                <mesh filename="package://agx_arm_description/agx_arm_urdf/nero/meshes/dae/gripper_link2.dae"/>
+                <mesh filename="package://agx_arm_urdf/nero/meshes/dae/gripper_link2.dae"/>
             </geometry>
         </visual>
@@ -78,5 +78,5 @@
             <origin xyz="0 0 0" rpy="0 0 0"/>
             <geometry>
-                <mesh filename="package://agx_arm_description/agx_arm_urdf/nero/meshes/gripper_link2.stl"/>
+                <mesh filename="package://agx_arm_urdf/nero/meshes/gripper_link2.stl"/>
             </geometry>
         </collision>

File: nero/urdf/nero_with_gripper_flange_description.xacro (robot description, xacro)
@@ -13,5 +13,5 @@
             <origin xyz="0 0 0" rpy="0 0 0"/>
             <geometry>
-                <mesh filename="package://agx_arm_description/agx_arm_urdf/nero/meshes/dae/gripper_flange.dae"/>
+                <mesh filename="package://agx_arm_urdf/nero/meshes/dae/gripper_flange.dae"/>
             </geometry>
         </visual>
@@ -19,5 +19,5 @@
             <origin xyz="0 0 0" rpy="0 0 0"/>
             <geometry>
-                <mesh filename="package://agx_arm_description/agx_arm_urdf/nero/meshes/gripper_flange.stl"/>
+                <mesh filename="package://agx_arm_urdf/nero/meshes/gripper_flange.stl"/>
             </geometry>
         </collision>

File: nero/urdf/nero_with_revo2_flange_description.xacro (robot description, xacro)
@@ -13,5 +13,5 @@
             <origin xyz="0 0 0" rpy="0 0 0"/>
             <geometry>
-                <mesh filename="package://agx_arm_description/agx_arm_urdf/nero/meshes/dae/revo2_flange.dae"/>
+                <mesh filename="package://agx_arm_urdf/nero/meshes/dae/revo2_flange.dae"/>
             </geometry>
         </visual>
@@ -19,5 +19,5 @@
             <origin xyz="0 0 0" rpy="0 0 0"/>
             <geometry>
-                <mesh filename="package://agx_arm_description/agx_arm_urdf/nero/meshes/revo2_flange.stl"/>
+                <mesh filename="package://agx_arm_urdf/nero/meshes/revo2_flange.stl"/>
             </geometry>
         </collision>

File: piper/urdf/piper_description.urdf (robot description, URDF)
Before this commit: robot piper, 8 links, 7 joints
Links:
- link base_link: geometry collision mesh filename=package://agx_arm_urdf/piper/meshes/base_link.stl; visual mesh filename=package://agx_arm_urdf/piper/meshes/dae/base_link.dae
- link link1: geometry collision mesh filename=package://agx_arm_urdf/piper/meshes/link1.stl; visual mesh filename=package://agx_arm_urdf/piper/meshes/dae/link1.dae
- link link2: geometry collision mesh filename=package://agx_arm_urdf/piper/meshes/link2.stl; visual mesh filename=package://agx_arm_urdf/piper/meshes/dae/link2.dae
- link link3: geometry collision mesh filename=package://agx_arm_urdf/piper/meshes/link3.stl; visual mesh filename=package://agx_arm_urdf/piper/meshes/dae/link3.dae
- link link4: geometry collision mesh filename=package://agx_arm_urdf/piper/meshes/link4.stl; visual mesh filename=package://agx_arm_urdf/piper/meshes/dae/link4.dae
- link link5: geometry collision mesh filename=package://agx_arm_urdf/piper/meshes/link5.stl; visual mesh filename=package://agx_arm_urdf/piper/meshes/dae/link5.dae
- link link6: geometry collision mesh filename=package://agx_arm_urdf/piper/meshes/link6.stl; visual mesh filename=package://agx_arm_urdf/piper/meshes/dae/link6.dae

File: piper/urdf/piper_with_gripper_description.xacro (robot description, xacro)
@@ -13,5 +13,5 @@
             <origin xyz="0 0 0" rpy="0 0 0"/>
             <geometry>
-                <mesh filename="package://agx_arm_description/agx_arm_urdf/piper/meshes/dae/flange.dae"/>
+                <mesh filename="package://agx_arm_urdf/piper/meshes/dae/flange.dae"/>
             </geometry>
         </visual>
@@ -19,5 +19,5 @@
             <origin xyz="0 0 0" rpy="0 0 0"/>
             <geometry>
-                <mesh filename="package://agx_arm_description/agx_arm_urdf/piper/meshes/flange.stl"/>
+                <mesh filename="package://agx_arm_urdf/piper/meshes/flange.stl"/>
             </geometry>
         </collision>
@@ -37,5 +37,5 @@
             <origin xyz="0 0 0" rpy="0 0 0"/>
             <geometry>
-                <mesh filename="package://agx_arm_description/agx_arm_urdf/piper/meshes/dae/gripper_base.dae"/>
+                <mesh filename="package://agx_arm_urdf/piper/meshes/dae/gripper_base.dae"/>
             </geometry>
         </visual>
@@ -43,5 +43,5 @@
             <origin xyz="0 0 0" rpy="0 0 0"/>
             <geometry>
-                <mesh filename="package://agx_arm_description/agx_arm_urdf/piper/meshes/gripper_base.stl"/>
+                <mesh filename="package://agx_arm_urdf/piper/meshes/gripper_base.stl"/>
             </geometry>
         </collision>
@@ -69,5 +69,5 @@
             <origin xyz="0 0 0" rpy="0 0 0"/>
             <geometry>
-                <mesh filename="package://agx_arm_description/agx_arm_urdf/piper/meshes/dae/gripper_link1.dae"/>
+                <mesh filename="package://agx_arm_urdf/piper/meshes/dae/gripper_link1.dae"/>
             </geometry>
         </visual>
@@ -75,5 +75,5 @@
             <origin xyz="0 0 0" rpy="0 0 0"/>
             <geometry>
-                <mesh filename="package://agx_arm_description/agx_arm_urdf/piper/meshes/gripper_link1.stl"/>
+                <mesh filename="package://agx_arm_urdf/piper/meshes/gripper_link1.stl"/>
             </geometry>
         </collision>
@@ -96,5 +96,5 @@
             <origin xyz="0 0 0" rpy="0 0 0"/>
             <geometry>
-                <mesh filename="package://agx_arm_description/agx_arm_urdf/piper/meshes/dae/gripper_link2.dae"/>
+                <mesh filename="package://agx_arm_urdf/piper/meshes/dae/gripper_link2.dae"/>
             </geometry>
         </visual>
@@ -102,5 +102,5 @@
             <origin xyz="0 0 0" rpy="0 0 0"/>
             <geometry>
-                <mesh filename="package://agx_arm_description/agx_arm_urdf/piper/meshes/gripper_link2.stl"/>
+                <mesh filename="package://agx_arm_urdf/piper/meshes/gripper_link2.stl"/>
             </geometry>
         </collision>

File: piper/urdf/piper_with_left_revo2_description.xacro (robot description, xacro)
@@ -15,5 +15,5 @@
             <origin xyz="0 0 0" rpy="0 0 0"/>
             <geometry>
-                <mesh filename="package://agx_arm_description/agx_arm_urdf/piper/meshes/dae/flange.dae"/>
+                <mesh filename="package://agx_arm_urdf/piper/meshes/dae/flange.dae"/>
             </geometry>
         </visual>
@@ -21,5 +21,5 @@
             <origin xyz="0 0 0" rpy="0 0 0"/>
             <geometry>
-                <mesh filename="package://agx_arm_description/agx_arm_urdf/piper/meshes/flange.stl"/>
+                <mesh filename="package://agx_arm_urdf/piper/meshes/flange.stl"/>
             </geometry>
         </collision>

File: piper/urdf/piper_with_right_revo2_description.xacro (robot description, xacro)
@@ -15,5 +15,5 @@
             <origin xyz="0 0 0" rpy="0 0 0"/>
             <geometry>
-                <mesh filename="package://agx_arm_description/agx_arm_urdf/piper/meshes/dae/flange.dae"/>
+                <mesh filename="package://agx_arm_urdf/piper/meshes/dae/flange.dae"/>
             </geometry>
         </visual>
@@ -21,5 +21,5 @@
             <origin xyz="0 0 0" rpy="0 0 0"/>
             <geometry>
-                <mesh filename="package://agx_arm_description/agx_arm_urdf/piper/meshes/flange.stl"/>
+                <mesh filename="package://agx_arm_urdf/piper/meshes/flange.stl"/>
             </geometry>
         </collision>

File: piper_h/urdf/piper_h_description.urdf (robot description, URDF)
Before this commit: robot piper_h, 8 links, 7 joints
Links:
- link base_link: geometry collision mesh filename=package://agx_arm_urdf/piper_h/meshes/base_link.stl; visual mesh filename=package://agx_arm_urdf/piper_h/meshes/dae/base_link.dae
- link link1: geometry collision mesh filename=package://agx_arm_urdf/piper_h/meshes/link1.stl; visual mesh filename=package://agx_arm_urdf/piper_h/meshes/dae/link1.dae
- link link2: geometry collision mesh filename=package://agx_arm_urdf/piper_h/meshes/link2.stl; visual mesh filename=package://agx_arm_urdf/piper_h/meshes/dae/link2.dae
- link link3: geometry collision mesh filename=package://agx_arm_urdf/piper_h/meshes/link3.stl; visual mesh filename=package://agx_arm_urdf/piper_h/meshes/dae/link3.dae
- link link4: geometry collision mesh filename=package://agx_arm_urdf/piper_h/meshes/link4.stl; visual mesh filename=package://agx_arm_urdf/piper_h/meshes/dae/link4.dae
- link link5: geometry collision mesh filename=package://agx_arm_urdf/piper_h/meshes/link5.stl; visual mesh filename=package://agx_arm_urdf/piper_h/meshes/dae/link5.dae
- link link6: geometry collision mesh filename=package://agx_arm_urdf/piper_h/meshes/link6.stl; visual mesh filename=package://agx_arm_urdf/piper_h/meshes/dae/link6.dae

File: piper_h/urdf/piper_h_with_gripper_description.xacro (robot description, xacro)
@@ -13,5 +13,5 @@
             <origin xyz="0 0 0" rpy="0 0 0"/>
             <geometry>
-                <mesh filename="package://agx_arm_description/agx_arm_urdf/piper_h/meshes/dae/flange.dae"/>
+                <mesh filename="package://agx_arm_urdf/piper_h/meshes/dae/flange.dae"/>
             </geometry>
         </visual>
@@ -19,5 +19,5 @@
             <origin xyz="0 0 0" rpy="0 0 0"/>
             <geometry>
-                <mesh filename="package://agx_arm_description/agx_arm_urdf/piper_h/meshes/flange.stl"/>
+                <mesh filename="package://agx_arm_urdf/piper_h/meshes/flange.stl"/>
             </geometry>
         </collision>
@@ -37,5 +37,5 @@
             <origin xyz="0 0 0" rpy="0 0 0"/>
             <geometry>
-                <mesh filename="package://agx_arm_description/agx_arm_urdf/piper_h/meshes/dae/gripper_base.dae"/>
+                <mesh filename="package://agx_arm_urdf/piper_h/meshes/dae/gripper_base.dae"/>
             </geometry>
         </visual>
@@ -43,5 +43,5 @@
             <origin xyz="0 0 0" rpy="0 0 0"/>
             <geometry>
-                <mesh filename="package://agx_arm_description/agx_arm_urdf/piper_h/meshes/gripper_base.stl"/>
+                <mesh filename="package://agx_arm_urdf/piper_h/meshes/gripper_base.stl"/>
             </geometry>
         </collision>
@@ -69,5 +69,5 @@
             <origin xyz="0 0 0" rpy="0 0 0"/>
             <geometry>
-                <mesh filename="package://agx_arm_description/agx_arm_urdf/piper_h/meshes/dae/gripper_link1.dae"/>
+                <mesh filename="package://agx_arm_urdf/piper_h/meshes/dae/gripper_link1.dae"/>
             </geometry>
         </visual>
@@ -75,5 +75,5 @@
             <origin xyz="0 0 0" rpy="0 0 0"/>
             <geometry>
-                <mesh filename="package://agx_arm_description/agx_arm_urdf/piper_h/meshes/gripper_link1.stl"/>
+                <mesh filename="package://agx_arm_urdf/piper_h/meshes/gripper_link1.stl"/>
             </geometry>
         </collision>
@@ -96,5 +96,5 @@
             <origin xyz="0 0 0" rpy="0 0 0"/>
             <geometry>
-                <mesh filename="package://agx_arm_description/agx_arm_urdf/piper_h/meshes/dae/gripper_link2.dae"/>
+                <mesh filename="package://agx_arm_urdf/piper_h/meshes/dae/gripper_link2.dae"/>
             </geometry>
         </visual>
@@ -102,5 +102,5 @@
             <origin xyz="0 0 0" rpy="0 0 0"/>
             <geometry>
-                <mesh filename="package://agx_arm_description/agx_arm_urdf/piper_h/meshes/gripper_link2.stl"/>
+                <mesh filename="package://agx_arm_urdf/piper_h/meshes/gripper_link2.stl"/>
             </geometry>
         </collision>

File: piper_h/urdf/piper_h_with_left_revo2_description.xacro (robot description, xacro)
@@ -15,5 +15,5 @@
             <origin xyz="0 0 0" rpy="0 0 0"/>
             <geometry>
-                <mesh filename="package://agx_arm_description/agx_arm_urdf/piper_h/meshes/dae/flange.dae"/>
+                <mesh filename="package://agx_arm_urdf/piper_h/meshes/dae/flange.dae"/>
             </geometry>
         </visual>
@@ -21,5 +21,5 @@
             <origin xyz="0 0 0" rpy="0 0 0"/>
             <geometry>
-                <mesh filename="package://agx_arm_description/agx_arm_urdf/piper_h/meshes/flange.stl"/>
+                <mesh filename="package://agx_arm_urdf/piper_h/meshes/flange.stl"/>
             </geometry>
         </collision>

File: piper_h/urdf/piper_h_with_right_revo2_description.xacro (robot description, xacro)
@@ -15,5 +15,5 @@
             <origin xyz="0 0 0" rpy="0 0 0"/>
             <geometry>
-                <mesh filename="package://agx_arm_description/agx_arm_urdf/piper_h/meshes/dae/flange.dae"/>
+                <mesh filename="package://agx_arm_urdf/piper_h/meshes/dae/flange.dae"/>
             </geometry>
         </visual>
@@ -21,5 +21,5 @@
             <origin xyz="0 0 0" rpy="0 0 0"/>
             <geometry>
-                <mesh filename="package://agx_arm_description/agx_arm_urdf/piper_h/meshes/flange.stl"/>
+                <mesh filename="package://agx_arm_urdf/piper_h/meshes/flange.stl"/>
             </geometry>
         </collision>

File: piper_l/urdf/piper_l_description.urdf (robot description, URDF)
Before this commit: robot piper_l, 8 links, 7 joints
Links:
- link base_link: geometry collision mesh filename=package://agx_arm_urdf/piper_l/meshes/base_link.stl; visual mesh filename=package://agx_arm_urdf/piper_l/meshes/dae/base_link.dae
- link link1: geometry collision mesh filename=package://agx_arm_urdf/piper_l/meshes/link1.stl; visual mesh filename=package://agx_arm_urdf/piper_l/meshes/dae/link1.dae
- link link2: geometry collision mesh filename=package://agx_arm_urdf/piper_l/meshes/link2.stl; visual mesh filename=package://agx_arm_urdf/piper_l/meshes/dae/link2.dae
- link link3: geometry collision mesh filename=package://agx_arm_urdf/piper_l/meshes/link3.stl; visual mesh filename=package://agx_arm_urdf/piper_l/meshes/dae/link3.dae
- link link4: geometry collision mesh filename=package://agx_arm_urdf/piper_l/meshes/link4.stl; visual mesh filename=package://agx_arm_urdf/piper_l/meshes/dae/link4.dae
- link link5: geometry collision mesh filename=package://agx_arm_urdf/piper_l/meshes/link5.stl; visual mesh filename=package://agx_arm_urdf/piper_l/meshes/dae/link5.dae
- link link6: geometry collision mesh filename=package://agx_arm_urdf/piper_l/meshes/link6.stl; visual mesh filename=package://agx_arm_urdf/piper_l/meshes/dae/link6.dae

File: piper_l/urdf/piper_l_with_gripper_description.xacro (robot description, xacro)
@@ -13,5 +13,5 @@
             <origin xyz="0 0 0" rpy="0 0 0"/>
             <geometry>
-                <mesh filename="package://agx_arm_description/agx_arm_urdf/piper_l/meshes/dae/flange.dae"/>
+                <mesh filename="package://agx_arm_urdf/piper_l/meshes/dae/flange.dae"/>
             </geometry>
         </visual>
@@ -19,5 +19,5 @@
             <origin xyz="0 0 0" rpy="0 0 0"/>
             <geometry>
-                <mesh filename="package://agx_arm_description/agx_arm_urdf/piper_l/meshes/flange.stl"/>
+                <mesh filename="package://agx_arm_urdf/piper_l/meshes/flange.stl"/>
             </geometry>
         </collision>
@@ -37,5 +37,5 @@
             <origin xyz="0 0 0" rpy="0 0 0"/>
             <geometry>
-                <mesh filename="package://agx_arm_description/agx_arm_urdf/piper_l/meshes/dae/gripper_base.dae"/>
+                <mesh filename="package://agx_arm_urdf/piper_l/meshes/dae/gripper_base.dae"/>
             </geometry>
         </visual>
@@ -43,5 +43,5 @@
             <origin xyz="0 0 0" rpy="0 0 0"/>
             <geometry>
-                <mesh filename="package://agx_arm_description/agx_arm_urdf/piper_l/meshes/gripper_base.stl"/>
+                <mesh filename="package://agx_arm_urdf/piper_l/meshes/gripper_base.stl"/>
             </geometry>
         </collision>
@@ -69,5 +69,5 @@
             <origin xyz="0 0 0" rpy="0 0 0"/>
             <geometry>
-                <mesh filename="package://agx_arm_description/agx_arm_urdf/piper_l/meshes/dae/gripper_link1.dae"/>
+                <mesh filename="package://agx_arm_urdf/piper_l/meshes/dae/gripper_link1.dae"/>
             </geometry>
         </visual>
@@ -75,5 +75,5 @@
             <origin xyz="0 0 0" rpy="0 0 0"/>
             <geometry>
-                <mesh filename="package://agx_arm_description/agx_arm_urdf/piper_l/meshes/gripper_link1.stl"/>
+                <mesh filename="package://agx_arm_urdf/piper_l/meshes/gripper_link1.stl"/>
             </geometry>
         </collision>
@@ -96,5 +96,5 @@
             <origin xyz="0 0 0" rpy="0 0 0"/>
             <geometry>
-                <mesh filename="package://agx_arm_description/agx_arm_urdf/piper_l/meshes/dae/gripper_link2.dae"/>
+                <mesh filename="package://agx_arm_urdf/piper_l/meshes/dae/gripper_link2.dae"/>
             </geometry>
         </visual>
@@ -102,5 +102,5 @@
             <origin xyz="0 0 0" rpy="0 0 0"/>
             <geometry>
-                <mesh filename="package://agx_arm_description/agx_arm_urdf/piper_l/meshes/gripper_link2.stl"/>
+                <mesh filename="package://agx_arm_urdf/piper_l/meshes/gripper_link2.stl"/>
             </geometry>
         </collision>

File: piper_l/urdf/piper_l_with_left_revo2_description.xacro (robot description, xacro)
@@ -15,5 +15,5 @@
             <origin xyz="0 0 0" rpy="0 0 0"/>
             <geometry>
-                <mesh filename="package://agx_arm_description/agx_arm_urdf/piper_l/meshes/dae/flange.dae"/>
+                <mesh filename="package://agx_arm_urdf/piper_l/meshes/dae/flange.dae"/>
             </geometry>
         </visual>
@@ -21,5 +21,5 @@
             <origin xyz="0 0 0" rpy="0 0 0"/>
             <geometry>
-                <mesh filename="package://agx_arm_description/agx_arm_urdf/piper_l/meshes/flange.stl"/>
+                <mesh filename="package://agx_arm_urdf/piper_l/meshes/flange.stl"/>
             </geometry>
         </collision>

File: piper_l/urdf/piper_l_with_right_revo2_description.xacro (robot description, xacro)
@@ -15,5 +15,5 @@
             <origin xyz="0 0 0" rpy="0 0 0"/>
             <geometry>
-                <mesh filename="package://agx_arm_description/agx_arm_urdf/piper_l/meshes/dae/flange.dae"/>
+                <mesh filename="package://agx_arm_urdf/piper_l/meshes/dae/flange.dae"/>
             </geometry>
         </visual>
@@ -21,5 +21,5 @@
             <origin xyz="0 0 0" rpy="0 0 0"/>
             <geometry>
-                <mesh filename="package://agx_arm_description/agx_arm_urdf/piper_l/meshes/flange.stl"/>
+                <mesh filename="package://agx_arm_urdf/piper_l/meshes/flange.stl"/>
             </geometry>
         </collision>
