Commit message: feat: make agx_arm_urdf a standalone ROS 2 package
- add ament_cmake package metadata
- add a prefix-aware Piper Xacro macro
- update mesh URIs to resolve from agx_arm_urdf
- document standalone and vcstool-based usage

File: piper_x/urdf/piper_x_description.urdf (robot description, URDF)
Before this commit: robot piper_x, 8 links, 7 joints
Links:
- link base_link: geometry collision mesh filename=package://agx_arm_urdf/piper_x/meshes/base_link.stl; visual mesh filename=package://agx_arm_urdf/piper_x/meshes/dae/base_link.dae
- link link1: geometry collision mesh filename=package://agx_arm_urdf/piper_x/meshes/link1.stl; visual mesh filename=package://agx_arm_urdf/piper_x/meshes/dae/link1.dae
- link link2: geometry collision mesh filename=package://agx_arm_urdf/piper_x/meshes/link2.stl; visual mesh filename=package://agx_arm_urdf/piper_x/meshes/dae/link2.dae
- link link3: geometry collision mesh filename=package://agx_arm_urdf/piper_x/meshes/link3.stl; visual mesh filename=package://agx_arm_urdf/piper_x/meshes/dae/link3.dae
- link link4: geometry collision mesh filename=package://agx_arm_urdf/piper_x/meshes/link4.stl; visual mesh filename=package://agx_arm_urdf/piper_x/meshes/dae/link4.dae
- link link5: geometry collision mesh filename=package://agx_arm_urdf/piper_x/meshes/link5.stl; visual mesh filename=package://agx_arm_urdf/piper_x/meshes/dae/link5.dae
- link link6: geometry collision mesh filename=package://agx_arm_urdf/piper_x/meshes/link6.stl; visual mesh filename=package://agx_arm_urdf/piper_x/meshes/dae/link6.dae

File: piper_x/urdf/piper_x_with_gripper_description.xacro (robot description, xacro)
@@ -13,5 +13,5 @@
             <origin xyz="0 0 0" rpy="0 0 0"/>
             <geometry>
-                <mesh filename="package://agx_arm_description/agx_arm_urdf/piper_x/meshes/dae/flange.dae"/>
+                <mesh filename="package://agx_arm_urdf/piper_x/meshes/dae/flange.dae"/>
             </geometry>
         </visual>
@@ -19,5 +19,5 @@
             <origin xyz="0 0 0" rpy="0 0 0"/>
             <geometry>
-                <mesh filename="package://agx_arm_description/agx_arm_urdf/piper_x/meshes/flange.stl"/>
+                <mesh filename="package://agx_arm_urdf/piper_x/meshes/flange.stl"/>
             </geometry>
         </collision>
@@ -37,5 +37,5 @@
             <origin xyz="0 0 0" rpy="0 0 0"/>
             <geometry>
-                <mesh filename="package://agx_arm_description/agx_arm_urdf/piper_x/meshes/dae/gripper_base.dae"/>
+                <mesh filename="package://agx_arm_urdf/piper_x/meshes/dae/gripper_base.dae"/>
             </geometry>
         </visual>
@@ -43,5 +43,5 @@
             <origin xyz="0 0 0" rpy="0 0 0"/>
             <geometry>
-                <mesh filename="package://agx_arm_description/agx_arm_urdf/piper_x/meshes/gripper_base.stl"/>
+                <mesh filename="package://agx_arm_urdf/piper_x/meshes/gripper_base.stl"/>
             </geometry>
         </collision>
@@ -69,5 +69,5 @@
             <origin xyz="0 0 0" rpy="0 0 0"/>
             <geometry>
-                <mesh filename="package://agx_arm_description/agx_arm_urdf/piper_x/meshes/dae/gripper_link1.dae"/>
+                <mesh filename="package://agx_arm_urdf/piper_x/meshes/dae/gripper_link1.dae"/>
             </geometry>
         </visual>
@@ -75,5 +75,5 @@
             <origin xyz="0 0 0" rpy="0 0 0"/>
             <geometry>
-                <mesh filename="package://agx_arm_description/agx_arm_urdf/piper_x/meshes/gripper_link1.stl"/>
+                <mesh filename="package://agx_arm_urdf/piper_x/meshes/gripper_link1.stl"/>
             </geometry>
         </collision>
@@ -96,5 +96,5 @@
             <origin xyz="0 0 0" rpy="0 0 0"/>
             <geometry>
-                <mesh filename="package://agx_arm_description/agx_arm_urdf/piper_x/meshes/dae/gripper_link2.dae"/>
+                <mesh filename="package://agx_arm_urdf/piper_x/meshes/dae/gripper_link2.dae"/>
             </geometry>
         </visual>
@@ -102,5 +102,5 @@
             <origin xyz="0 0 0" rpy="0 0 0"/>
             <geometry>
-                <mesh filename="package://agx_arm_description/agx_arm_urdf/piper_x/meshes/gripper_link2.stl"/>
+                <mesh filename="package://agx_arm_urdf/piper_x/meshes/gripper_link2.stl"/>
             </geometry>
         </collision>

File: piper_x/urdf/piper_x_with_left_revo2_description.xacro (robot description, xacro)
@@ -15,5 +15,5 @@
             <origin xyz="0 0 0" rpy="0 0 0"/>
             <geometry>
-                <mesh filename="package://agx_arm_description/agx_arm_urdf/piper_x/meshes/dae/flange.dae"/>
+                <mesh filename="package://agx_arm_urdf/piper_x/meshes/dae/flange.dae"/>
             </geometry>
         </visual>
@@ -21,5 +21,5 @@
             <origin xyz="0 0 0" rpy="0 0 0"/>
             <geometry>
-                <mesh filename="package://agx_arm_description/agx_arm_urdf/piper_x/meshes/flange.stl"/>
+                <mesh filename="package://agx_arm_urdf/piper_x/meshes/flange.stl"/>
             </geometry>
         </collision>

File: piper_x/urdf/piper_x_with_right_revo2_description.xacro (robot description, xacro)
@@ -15,5 +15,5 @@
             <origin xyz="0 0 0" rpy="0 0 0"/>
             <geometry>
-                <mesh filename="package://agx_arm_description/agx_arm_urdf/piper_x/meshes/dae/flange.dae"/>
+                <mesh filename="package://agx_arm_urdf/piper_x/meshes/dae/flange.dae"/>
             </geometry>
         </visual>
@@ -21,5 +21,5 @@
             <origin xyz="0 0 0" rpy="0 0 0"/>
             <geometry>
-                <mesh filename="package://agx_arm_description/agx_arm_urdf/piper_x/meshes/flange.stl"/>
+                <mesh filename="package://agx_arm_urdf/piper_x/meshes/flange.stl"/>
             </geometry>
         </collision>
