Commit message: corrected broken path, add gripper_tcp to piper_H

File: nero/urdf/nero_with_gripper_description.xacro (robot description, xacro)
@@ -3,5 +3,5 @@
      For more information, please see http://wiki.ros.org/sw_urdf_exporter -->
 <robot xmlns:xacro="http://www.ros.org/wiki/xacro" name="nero">
-<xacro:include filename="$(find agx_arm_description)/agx_arm_urdf/nero/urdf/nero_with_gripper_flange_description.xacro"/>
+<xacro:include filename="$(find agx_arm_urdf)/nero/urdf/nero_with_gripper_flange_description.xacro"/>
     <link name="gripper_base">
         <inertial>

File: nero/urdf/nero_with_gripper_flange_description.xacro (robot description, xacro)
@@ -3,5 +3,5 @@
      For more information, please see http://wiki.ros.org/sw_urdf_exporter -->
 <robot xmlns:xacro="http://www.ros.org/wiki/xacro" name="nero">
-<xacro:include filename="$(find agx_arm_description)/agx_arm_urdf/nero/urdf/nero_description.urdf"/>
+<xacro:include filename="$(find agx_arm_urdf)/nero/urdf/nero_description.urdf"/>
     <link name="gripper_flange">
         <inertial>

File: nero/urdf/nero_with_left_revo2_description.xacro (robot description, xacro)
@@ -4,6 +4,6 @@
      For more information, please see http://wiki.ros.org/sw_urdf_exporter -->
 <robot xmlns:xacro="http://www.ros.org/wiki/xacro" name="nero">
-<xacro:include filename="$(find agx_arm_description)/agx_arm_urdf/revo2/urdf/revo2_left_hand.urdf"/>
-<xacro:include filename="$(find agx_arm_description)/agx_arm_urdf/nero/urdf/nero_with_revo2_flange_description.xacro"/>
+<xacro:include filename="$(find agx_arm_urdf)/revo2/urdf/revo2_left_hand.urdf"/>
+<xacro:include filename="$(find agx_arm_urdf)/nero/urdf/nero_with_revo2_flange_description.xacro"/>
     <joint name="hand_base_joint" type="fixed">
         <origin xyz="0.0 0.0 0.012" rpy="0 0 3.1415926"/>

File: nero/urdf/nero_with_revo2_flange_description.xacro (robot description, xacro)
@@ -3,5 +3,5 @@
      For more information, please see http://wiki.ros.org/sw_urdf_exporter -->
 <robot xmlns:xacro="http://www.ros.org/wiki/xacro" name="nero">
-<xacro:include filename="$(find agx_arm_description)/agx_arm_urdf/nero/urdf/nero_description.urdf"/>
+<xacro:include filename="$(find agx_arm_urdf)/nero/urdf/nero_description.urdf"/>
     <link name="revo2_flange">
         <inertial>

File: nero/urdf/nero_with_right_revo2_description.xacro (robot description, xacro)
@@ -4,6 +4,6 @@
      For more information, please see http://wiki.ros.org/sw_urdf_exporter -->
 <robot xmlns:xacro="http://www.ros.org/wiki/xacro" name="nero">
-<xacro:include filename="$(find agx_arm_description)/agx_arm_urdf/revo2/urdf/revo2_right_hand.urdf"/>
-<xacro:include filename="$(find agx_arm_description)/agx_arm_urdf/nero/urdf/nero_with_revo2_flange_description.xacro"/>
+<xacro:include filename="$(find agx_arm_urdf)/revo2/urdf/revo2_right_hand.urdf"/>
+<xacro:include filename="$(find agx_arm_urdf)/nero/urdf/nero_with_revo2_flange_description.xacro"/>
     <joint name="hand_base_joint" type="fixed">
         <origin xyz="0.0 0.0 0.012" rpy="0 0 3.1415926"/>

File: piper/urdf/piper_with_gripper_description.xacro (robot description, xacro)
@@ -3,5 +3,5 @@
      For more information, please see http://wiki.ros.org/sw_urdf_exporter -->
 <robot xmlns:xacro="http://www.ros.org/wiki/xacro" name="piper">
-<xacro:include filename="$(find agx_arm_description)/agx_arm_urdf/piper/urdf/piper_description.urdf"/>
+<xacro:include filename="$(find agx_arm_urdf)/piper/urdf/piper_description.urdf"/>
     <link name="flange_link">
         <inertial>

File: piper/urdf/piper_with_left_revo2_description.xacro (robot description, xacro)
@@ -4,6 +4,6 @@
      For more information, please see http://wiki.ros.org/sw_urdf_exporter -->
 <robot xmlns:xacro="http://www.ros.org/wiki/xacro" name="piper">
-<xacro:include filename="$(find agx_arm_description)/agx_arm_urdf/revo2/urdf/revo2_left_hand.urdf"/>
-<xacro:include filename="$(find agx_arm_description)/agx_arm_urdf/piper/urdf/piper_description.urdf"/>
+<xacro:include filename="$(find agx_arm_urdf)/revo2/urdf/revo2_left_hand.urdf"/>
+<xacro:include filename="$(find agx_arm_urdf)/piper/urdf/piper_description.urdf"/>
     <link name="flange_link">
         <inertial>

File: piper/urdf/piper_with_right_revo2_description.xacro (robot description, xacro)
@@ -4,6 +4,6 @@
      For more information, please see http://wiki.ros.org/sw_urdf_exporter -->
 <robot xmlns:xacro="http://www.ros.org/wiki/xacro" name="piper">
-<xacro:include filename="$(find agx_arm_description)/agx_arm_urdf/revo2/urdf/revo2_right_hand.urdf"/>
-<xacro:include filename="$(find agx_arm_description)/agx_arm_urdf/piper/urdf/piper_description.urdf"/>
+<xacro:include filename="$(find agx_arm_urdf)/revo2/urdf/revo2_right_hand.urdf"/>
+<xacro:include filename="$(find agx_arm_urdf)/piper/urdf/piper_description.urdf"/>
     <link name="flange_link">
         <inertial>

File: piper_h/urdf/piper_h_with_gripper_description.xacro (robot description, xacro)
@@ -3,5 +3,5 @@
      For more information, please see http://wiki.ros.org/sw_urdf_exporter -->
 <robot xmlns:xacro="http://www.ros.org/wiki/xacro" name="piper_h">
-<xacro:include filename="$(find agx_arm_description)/agx_arm_urdf/piper_h/urdf/piper_h_description.urdf"/>
+<xacro:include filename="$(find agx_arm_urdf)/piper_h/urdf/piper_h_description.urdf"/>
     <link name="flange_link">
         <inertial>
@@ -51,4 +51,10 @@
         <parent link="flange_link"/>
         <child link="gripper_base"/>
+    </joint>
+    <link name="gripper_tcp"/>
+    <joint name="gripper_tcp_joint" type="fixed">
+        <origin xyz="0 0 0.138" rpy="0 0 0"/>
+        <parent link="gripper_base"/>
+        <child link="gripper_tcp"/>
     </joint>
     <link name="gripper_link"/>

File: piper_h/urdf/piper_h_with_left_revo2_description.xacro (robot description, xacro)
@@ -4,6 +4,6 @@
      For more information, please see http://wiki.ros.org/sw_urdf_exporter -->
 <robot xmlns:xacro="http://www.ros.org/wiki/xacro" name="piper_h">
-<xacro:include filename="$(find agx_arm_description)/agx_arm_urdf/revo2/urdf/revo2_left_hand.urdf"/>
-<xacro:include filename="$(find agx_arm_description)/agx_arm_urdf/piper_h/urdf/piper_h_description.urdf"/>
+<xacro:include filename="$(find agx_arm_urdf)/revo2/urdf/revo2_left_hand.urdf"/>
+<xacro:include filename="$(find agx_arm_urdf)/piper_h/urdf/piper_h_description.urdf"/>
     <link name="flange_link">
         <inertial>

File: piper_h/urdf/piper_h_with_right_revo2_description.xacro (robot description, xacro)
@@ -4,6 +4,6 @@
      For more information, please see http://wiki.ros.org/sw_urdf_exporter -->
 <robot xmlns:xacro="http://www.ros.org/wiki/xacro" name="piper_h">
-<xacro:include filename="$(find agx_arm_description)/agx_arm_urdf/revo2/urdf/revo2_right_hand.urdf"/>
-<xacro:include filename="$(find agx_arm_description)/agx_arm_urdf/piper_h/urdf/piper_h_description.urdf"/>
+<xacro:include filename="$(find agx_arm_urdf)/revo2/urdf/revo2_right_hand.urdf"/>
+<xacro:include filename="$(find agx_arm_urdf)/piper_h/urdf/piper_h_description.urdf"/>
     <link name="flange_link">
         <inertial>

File: piper_l/urdf/piper_l_with_gripper_description.xacro (robot description, xacro)
@@ -3,5 +3,5 @@
      For more information, please see http://wiki.ros.org/sw_urdf_exporter -->
 <robot xmlns:xacro="http://www.ros.org/wiki/xacro" name="piper_l">
-<xacro:include filename="$(find agx_arm_description)/agx_arm_urdf/piper_l/urdf/piper_l_description.urdf"/>
+<xacro:include filename="$(find agx_arm_urdf)/piper_l/urdf/piper_l_description.urdf"/>
     <link name="flange_link">
         <inertial>

File: piper_l/urdf/piper_l_with_left_revo2_description.xacro (robot description, xacro)
@@ -4,6 +4,6 @@
      For more information, please see http://wiki.ros.org/sw_urdf_exporter -->
 <robot xmlns:xacro="http://www.ros.org/wiki/xacro" name="piper_l">
-<xacro:include filename="$(find agx_arm_description)/agx_arm_urdf/revo2/urdf/revo2_left_hand.urdf"/>
-<xacro:include filename="$(find agx_arm_description)/agx_arm_urdf/piper_l/urdf/piper_l_description.urdf"/>
+<xacro:include filename="$(find agx_arm_urdf)/revo2/urdf/revo2_left_hand.urdf"/>
+<xacro:include filename="$(find agx_arm_urdf)/piper_l/urdf/piper_l_description.urdf"/>
     <link name="flange_link">
         <inertial>

File: piper_l/urdf/piper_l_with_right_revo2_description.xacro (robot description, xacro)
@@ -4,6 +4,6 @@
      For more information, please see http://wiki.ros.org/sw_urdf_exporter -->
 <robot xmlns:xacro="http://www.ros.org/wiki/xacro" name="piper_l">
-<xacro:include filename="$(find agx_arm_description)/agx_arm_urdf/revo2/urdf/revo2_right_hand.urdf"/>
-<xacro:include filename="$(find agx_arm_description)/agx_arm_urdf/piper_l/urdf/piper_l_description.urdf"/>
+<xacro:include filename="$(find agx_arm_urdf)/revo2/urdf/revo2_right_hand.urdf"/>
+<xacro:include filename="$(find agx_arm_urdf)/piper_l/urdf/piper_l_description.urdf"/>
     <link name="flange_link">
         <inertial>

File: piper_x/urdf/piper_x_with_gripper_description.xacro (robot description, xacro)
@@ -3,5 +3,5 @@
      For more information, please see http://wiki.ros.org/sw_urdf_exporter -->
 <robot xmlns:xacro="http://www.ros.org/wiki/xacro" name="piper_x">
-<xacro:include filename="$(find agx_arm_description)/agx_arm_urdf/piper_x/urdf/piper_x_description.urdf"/>
+<xacro:include filename="$(find agx_arm_urdf)/piper_x/urdf/piper_x_description.urdf"/>
     <link name="flange_link">
         <inertial>

File: piper_x/urdf/piper_x_with_left_revo2_description.xacro (robot description, xacro)
@@ -4,6 +4,6 @@
      For more information, please see http://wiki.ros.org/sw_urdf_exporter -->
 <robot xmlns:xacro="http://www.ros.org/wiki/xacro" name="piper_x">
-<xacro:include filename="$(find agx_arm_description)/agx_arm_urdf/revo2/urdf/revo2_left_hand.urdf"/>
-<xacro:include filename="$(find agx_arm_description)/agx_arm_urdf/piper_x/urdf/piper_x_description.urdf"/>
+<xacro:include filename="$(find agx_arm_urdf)/revo2/urdf/revo2_left_hand.urdf"/>
+<xacro:include filename="$(find agx_arm_urdf)/piper_x/urdf/piper_x_description.urdf"/>
     <link name="flange_link">
         <inertial>

File: piper_x/urdf/piper_x_with_right_revo2_description.xacro (robot description, xacro)
@@ -4,6 +4,6 @@
      For more information, please see http://wiki.ros.org/sw_urdf_exporter -->
 <robot xmlns:xacro="http://www.ros.org/wiki/xacro" name="piper_x">
-<xacro:include filename="$(find agx_arm_description)/agx_arm_urdf/revo2/urdf/revo2_right_hand.urdf"/>
-<xacro:include filename="$(find agx_arm_description)/agx_arm_urdf/piper_x/urdf/piper_x_description.urdf"/>
+<xacro:include filename="$(find agx_arm_urdf)/revo2/urdf/revo2_right_hand.urdf"/>
+<xacro:include filename="$(find agx_arm_urdf)/piper_x/urdf/piper_x_description.urdf"/>
     <link name="flange_link">
         <inertial>

Commit message: add gripper_tcp frame to other robots

File: nero/urdf/nero_with_gripper_description.xacro (robot description, xacro)
@@ -27,4 +27,10 @@
         <parent link="gripper_flange"/>
         <child link="gripper_base"/>
+    </joint>
+    <link name="gripper_tcp"/>
+    <joint name="gripper_tcp_joint" type="fixed">
+        <origin xyz="0 0 0.138" rpy="0 0 0"/>
+        <parent link="gripper_base"/>
+        <child link="gripper_tcp"/>
     </joint>
     <link name="gripper_link"/>

File: piper/urdf/piper_with_gripper_description.xacro (robot description, xacro)
@@ -51,4 +51,10 @@
         <parent link="flange_link"/>
         <child link="gripper_base"/>
+    </joint>
+    <link name="gripper_tcp"/>
+    <joint name="gripper_tcp_joint" type="fixed">
+        <origin xyz="0 0 0.138" rpy="0 0 0"/>
+        <parent link="gripper_base"/>
+        <child link="gripper_tcp"/>
     </joint>
     <link name="gripper_link"/>

File: piper_l/urdf/piper_l_with_gripper_description.xacro (robot description, xacro)
@@ -51,4 +51,10 @@
         <parent link="flange_link"/>
         <child link="gripper_base"/>
+    </joint>
+    <link name="gripper_tcp"/>
+    <joint name="gripper_tcp_joint" type="fixed">
+        <origin xyz="0 0 0.138" rpy="0 0 0"/>
+        <parent link="gripper_base"/>
+        <child link="gripper_tcp"/>
     </joint>
     <link name="gripper_link"/>

File: piper_x/urdf/piper_x_with_gripper_description.xacro (robot description, xacro)
@@ -51,4 +51,10 @@
         <parent link="flange_link"/>
         <child link="gripper_base"/>
+    </joint>
+    <link name="gripper_tcp"/>
+    <joint name="gripper_tcp_joint" type="fixed">
+        <origin xyz="0 0 0.138" rpy="0 0 0"/>
+        <parent link="gripper_base"/>
+        <child link="gripper_tcp"/>
     </joint>
     <link name="gripper_link"/>
