Commit message: prefix for *_gripper arms + separate xacro for the gripper

File: nero/urdf/nero_with_gripper_description.xacro (robot description, xacro)
@@ -1,98 +1,12 @@
-<!-- This URDF was automatically created by SolidWorks to URDF Exporter! Originally created by Stephen Brawner (brawner@gmail.com)
-     Commit Version: 1.6.0-4-g7f85cfe  Build Version: 1.6.7995.38578
-     For more information, please see http://wiki.ros.org/sw_urdf_exporter -->
+<?xml version="1.0"?>
 <robot xmlns:xacro="http://www.ros.org/wiki/xacro" name="nero">
-<xacro:include filename="$(find agx_arm_urdf)/nero/urdf/nero_with_gripper_flange_description.xacro"/>
-    <link name="gripper_base">
-        <inertial>
-            <origin xyz="-0.000183807162235591 8.05033155577911E-05 0.0321436689908876" rpy="0 0 0"/>
-            <mass value="0.45"/>
-            <inertia ixx="0.00092934" ixy="0.00000034" ixz="-0.00000738" iyy="0.00071447" iyz="0.00000005" izz="0.00039442"/>
-        </inertial>
-        <visual>
-            <origin xyz="0 0 0" rpy="0 0 0"/>
-            <geometry>
-                <mesh filename="package://agx_arm_urdf/nero/meshes/dae/gripper_base.dae"/>
-            </geometry>
-        </visual>
-        <collision>
-            <origin xyz="0 0 0" rpy="0 0 0"/>
-            <geometry>
-                <mesh filename="package://agx_arm_urdf/nero/meshes/gripper_base.stl"/>
-            </geometry>
-        </collision>
-    </link>
-    <joint name="gripper_base_joint" type="fixed">
-        <origin xyz="0 0 0.006" rpy="0 0 0"/>
-        <parent link="gripper_flange"/>
-        <child link="gripper_base"/>
-    </joint>
-    <link name="gripper_tcp"/>
-    <joint name="gripper_tcp_joint" type="fixed">
-        <origin xyz="0 0 0.138" rpy="0 0 0"/>
-        <parent link="gripper_base"/>
-        <child link="gripper_tcp"/>
-    </joint>
-    <link name="gripper_link"/>
-    <joint name="gripper" type="prismatic">
-        <origin xyz="0 0 0" rpy="0 0 0"/>
-        <parent link="gripper_base"/>
-        <child link="gripper_link"/>
-        <axis xyz="0 0 1"/>
-        <limit lower="0" upper="0.1" effort="10" velocity="3"/>
-    </joint>
-    <link name="gripper_link1">
-        <inertial>
-            <origin xyz="0.00065123185041968 -0.0491929869131989 0.00972258769184025" rpy="0 0 0"/>
-            <mass value="0.025"/>
-            <inertia ixx="0.00007371" ixy="-0.00000113" ixz="0.00000021" iyy="0.00000781" iyz="-0.00001372" izz="0.0000747"/>
-        </inertial>
-        <visual>
-            <origin xyz="0 0 0" rpy="0 0 0"/>
-            <geometry>
-                <mesh filename="package://agx_arm_urdf/nero/meshes/dae/gripper_link1.dae"/>
-            </geometry>
-        </visual>
-        <collision>
-            <origin xyz="0 0 0" rpy="0 0 0"/>
-            <geometry>
-                <mesh filename="package://agx_arm_urdf/nero/meshes/gripper_link1.stl"/>
-            </geometry>
-        </collision>
-    </link>
-    <joint name="gripper_joint1" type="prismatic">
-        <origin xyz="0 0 0.138" rpy="1.5707963 0 3.1415926"/>
-        <parent link="gripper_base"/>
-        <child link="gripper_link1"/>
-        <axis xyz="0 0 1"/>
-        <limit lower="0" upper="0.05" effort="10" velocity="3"/>
-        <mimic joint="gripper" multiplier="0.5" offset="0.0"/>
-    </joint>
-    <link name="gripper_link2">
-        <inertial>
-            <origin xyz="0.00065123185041968 -0.0491929869131989 0.00972258769184025" rpy="0 0 0"/>
-            <mass value="0.025"/>
-            <inertia ixx="0.00007371" ixy="-0.00000113" ixz="0.00000021" iyy="0.00000781" iyz="-0.00001372" izz="0.0000747"/>
-        </inertial>
-        <visual>
-            <origin xyz="0 0 0" rpy="0 0 0"/>
-            <geometry>
-                <mesh filename="package://agx_arm_urdf/nero/meshes/dae/gripper_link2.dae"/>
-            </geometry>
-        </visual>
-        <collision>
-            <origin xyz="0 0 0" rpy="0 0 0"/>
-            <geometry>
-                <mesh filename="package://agx_arm_urdf/nero/meshes/gripper_link2.stl"/>
-            </geometry>
-        </collision>
-    </link>
-    <joint name="gripper_joint2" type="prismatic">
-        <origin xyz="0 0 0.138" rpy="1.5707963 0 0"/>
-        <parent link="gripper_base"/>
-        <child link="gripper_link2"/>
-        <axis xyz="0 0 -1"/>
-        <limit lower="-0.05" upper="0" effort="10" velocity="3"/>
-        <mimic joint="gripper" multiplier="-0.5" offset="0.0"/>
-    </joint>
+  <xacro:arg name="prefix" default=""/>
+  <xacro:include filename="$(find agx_arm_urdf)/nero/urdf/nero_with_gripper.xacro"/>
+  <xacro:nero_with_gripper prefix="$(arg prefix)"/>
+  <link name="world"/>
+  <joint name="world_to_$(arg prefix)base_link" type="fixed">
+    <parent link="world"/>
+    <child link="$(arg prefix)base_link"/>
+    <origin xyz="0 0 0" rpy="0 0 0"/>
+  </joint>
 </robot>

File: nero/urdf/nero_with_gripper_flange_description.xacro (robot description, xacro)
@@ -1,30 +1,12 @@
-<!-- This URDF was automatically created by SolidWorks to URDF Exporter! Originally created by Stephen Brawner (brawner@gmail.com)
-     Commit Version: 1.6.0-4-g7f85cfe  Build Version: 1.6.7995.38578
-     For more information, please see http://wiki.ros.org/sw_urdf_exporter -->
+<?xml version="1.0"?>
 <robot xmlns:xacro="http://www.ros.org/wiki/xacro" name="nero">
-<xacro:include filename="$(find agx_arm_urdf)/nero/urdf/nero_description.urdf"/>
-    <link name="gripper_flange">
-        <inertial>
-            <origin xyz="0.000253201 -0.000322696 -0.010082901" rpy="0 0 0"/>
-            <mass value="0.04771096"/>
-            <inertia ixx="36.14107e-06" ixy="0" ixz="0" iyy="17.824164e-06" iyz="0" izz="26.95944e-06"/>
-        </inertial>
-        <visual>
-            <origin xyz="0 0 0" rpy="0 0 0"/>
-            <geometry>
-                <mesh filename="package://agx_arm_urdf/nero/meshes/dae/gripper_flange.dae"/>
-            </geometry>
-        </visual>
-        <collision>
-            <origin xyz="0 0 0" rpy="0 0 0"/>
-            <geometry>
-                <mesh filename="package://agx_arm_urdf/nero/meshes/gripper_flange.stl"/>
-            </geometry>
-        </collision>
-    </link>
-    <joint name="gripper_flange_joint" type="fixed">
-        <origin xyz="0.031 0 -0.0235" rpy="-1.5708 0 -1.5708"/>
-        <parent link="link7"/>
-        <child link="gripper_flange"/>
-    </joint>
+  <xacro:arg name="prefix" default=""/>
+  <xacro:include filename="$(find agx_arm_urdf)/nero/urdf/nero_with_gripper.xacro"/>
+  <xacro:nero_with_gripper_flange prefix="$(arg prefix)"/>
+  <link name="world"/>
+  <joint name="world_to_$(arg prefix)base_link" type="fixed">
+    <parent link="world"/>
+    <child link="$(arg prefix)base_link"/>
+    <origin xyz="0 0 0" rpy="0 0 0"/>
+  </joint>
 </robot>

File: piper/urdf/piper_with_gripper_description.xacro (robot description, xacro)
@@ -1,122 +1,13 @@
-<!-- This URDF was automatically created by SolidWorks to URDF Exporter! Originally created by Stephen Brawner (brawner@gmail.com)
-     Commit Version: 1.6.0-4-g7f85cfe  Build Version: 1.6.7995.38578
-     For more information, please see http://wiki.ros.org/sw_urdf_exporter -->
+<?xml version="1.0"?>
 <robot xmlns:xacro="http://www.ros.org/wiki/xacro" name="piper">
-<xacro:include filename="$(find agx_arm_urdf)/piper/urdf/piper_description.urdf"/>
-    <link name="flange_link">
-        <inertial>
-            <origin xyz="1.151691e-03 0.782428e-03 4.798051e-03" rpy="0 0 0"/>
-            <mass value="0.04"/>
-            <inertia ixx="9.935389e-06" ixy="0.0" ixz="0.0" iyy="10.508003e-06" iyz="0.0" izz="19.652873e-06"/>
-        </inertial>
-        <visual>
-            <origin xyz="0 0 0" rpy="0 0 0"/>
-            <geometry>
-                <mesh filename="package://agx_arm_urdf/piper/meshes/dae/flange.dae"/>
-            </geometry>
-        </visual>
-        <collision>
-            <origin xyz="0 0 0" rpy="0 0 0"/>
-            <geometry>
-                <mesh filename="package://agx_arm_urdf/piper/meshes/flange.stl"/>
-            </geometry>
-        </collision>
-    </link>
-    <joint name="flange_joint" type="fixed">
-        <origin xyz="0 0 0" rpy="0 0 0"/>
-        <parent link="link6"/>
-        <child link="flange_link"/>
-    </joint>
-    <link name="gripper_base">
-        <inertial>
-            <origin xyz="-0.000183807162235591 8.05033155577911E-05 0.0321436689908876" rpy="0 0 0"/>
-            <mass value="0.45"/>
-            <inertia ixx="0.00092934" ixy="0.00000034" ixz="-0.00000738" iyy="0.00071447" iyz="0.00000005" izz="0.00039442"/>
-        </inertial>
-        <visual>
-            <origin xyz="0 0 0" rpy="0 0 0"/>
-            <geometry>
-                <mesh filename="package://agx_arm_urdf/piper/meshes/dae/gripper_base.dae"/>
-            </geometry>
-        </visual>
-        <collision>
-            <origin xyz="0 0 0" rpy="0 0 0"/>
-            <geometry>
-                <mesh filename="package://agx_arm_urdf/piper/meshes/gripper_base.stl"/>
-            </geometry>
-        </collision>
-    </link>
-    <joint name="gripper_base_joint" type="fixed">
-        <origin xyz="0 0 0.0045" rpy="0 0 0"/>
-        <parent link="flange_link"/>
-        <child link="gripper_base"/>
-    </joint>
-    <link name="gripper_tcp"/>
-    <joint name="gripper_tcp_joint" type="fixed">
-        <origin xyz="0 0 0.138" rpy="0 0 0"/>
-        <parent link="gripper_base"/>
-        <child link="gripper_tcp"/>
-    </joint>
-    <link name="gripper_link"/>
-    <joint name="gripper" type="prismatic">
-        <origin xyz="0 0 0" rpy="0 0 0"/>
-        <parent link="gripper_base"/>
-        <child link="gripper_link"/>
-        <axis xyz="0 0 1"/>
-        <limit lower="0" upper="0.1" effort="10" velocity="3"/>
-    </joint>
-    <link name="gripper_link1">
-        <inertial>
-            <origin xyz="0.00065123185041968 -0.0491929869131989 0.00972258769184025" rpy="0 0 0"/>
-            <mass value="0.025"/>
-            <inertia ixx="0.00007371" ixy="-0.00000113" ixz="0.00000021" iyy="0.00000781" iyz="-0.00001372" izz="0.0000747"/>
-        </inertial>
-        <visual>
-            <origin xyz="0 0 0" rpy="0 0 0"/>
-            <geometry>
-                <mesh filename="package://agx_arm_urdf/piper/meshes/dae/gripper_link1.dae"/>
-            </geometry>
-        </visual>
-        <collision>
-            <origin xyz="0 0 0" rpy="0 0 0"/>
-            <geometry>
-                <mesh filename="package://agx_arm_urdf/piper/meshes/gripper_link1.stl"/>
-            </geometry>
-        </collision>
-    </link>
-    <joint name="gripper_joint1" type="prismatic">
-        <origin xyz="0 0 0.138" rpy="1.5707963 0 0"/>
-        <parent link="gripper_base"/>
-        <child link="gripper_link1"/>
-        <axis xyz="0 0 1"/>
-        <limit lower="0" upper="0.05" effort="10" velocity="3"/>
-        <mimic joint="gripper" multiplier="0.5" offset="0.0"/>
-    </joint>
-    <link name="gripper_link2">
-        <inertial>
-            <origin xyz="0.00065123185041968 -0.0491929869131989 0.00972258769184025" rpy="0 0 0"/>
-            <mass value="0.025"/>
-            <inertia ixx="0.00007371" ixy="-0.00000113" ixz="0.00000021" iyy="0.00000781" iyz="-0.00001372" izz="0.0000747"/>
-        </inertial>
-        <visual>
-            <origin xyz="0 0 0" rpy="0 0 0"/>
-            <geometry>
-                <mesh filename="package://agx_arm_urdf/piper/meshes/dae/gripper_link2.dae"/>
-            </geometry>
-        </visual>
-        <collision>
-            <origin xyz="0 0 0" rpy="0 0 0"/>
-            <geometry>
-                <mesh filename="package://agx_arm_urdf/piper/meshes/gripper_link2.stl"/>
-            </geometry>
-        </collision>
-    </link>
-    <joint name="gripper_joint2" type="prismatic">
-        <origin xyz="0 0 0.138" rpy="1.5707963 0 -3.1415926"/>
-        <parent link="gripper_base"/>
-        <child link="gripper_link2"/>
-        <axis xyz="0 0 -1"/>
-        <limit lower="-0.05" upper="0" effort="10" velocity="3"/>
-        <mimic joint="gripper" multiplier="-0.5" offset="0.0"/>
-    </joint>
+  <xacro:arg name="prefix" default=""/>
+  <xacro:arg name="joint_limits_file" default="$(find agx_arm_urdf)/piper/config/joint_position_limits_original.yaml"/>
+  <xacro:include filename="$(find agx_arm_urdf)/piper/urdf/piper_with_gripper.xacro"/>
+  <xacro:piper_with_gripper prefix="$(arg prefix)" joint_limits_file="$(arg joint_limits_file)"/>
+  <link name="world"/>
+  <joint name="world_to_$(arg prefix)base_link" type="fixed">
+    <parent link="world"/>
+    <child link="$(arg prefix)base_link"/>
+    <origin xyz="0 0 0" rpy="0 0 0"/>
+  </joint>
 </robot>

File: piper_h/urdf/piper_h_with_gripper_description.xacro (robot description, xacro)
@@ -1,122 +1,12 @@
-<!-- This URDF was automatically created by SolidWorks to URDF Exporter! Originally created by Stephen Brawner (brawner@gmail.com)
-     Commit Version: 1.6.0-4-g7f85cfe  Build Version: 1.6.7995.38578
-     For more information, please see http://wiki.ros.org/sw_urdf_exporter -->
+<?xml version="1.0"?>
 <robot xmlns:xacro="http://www.ros.org/wiki/xacro" name="piper_h">
-<xacro:include filename="$(find agx_arm_urdf)/piper_h/urdf/piper_h_description.urdf"/>
-    <link name="flange_link">
-        <inertial>
-            <origin xyz="1.151691e-03 0.782428e-03 4.798051e-03" rpy="0 0 0"/>
-            <mass value="0.04"/>
-            <inertia ixx="9.935389e-06" ixy="0.0" ixz="0.0" iyy="10.508003e-06" iyz="0.0" izz="19.652873e-06"/>
-        </inertial>
-        <visual>
-            <origin xyz="0 0 0" rpy="0 0 0"/>
-            <geometry>
-                <mesh filename="package://agx_arm_urdf/piper_h/meshes/dae/flange.dae"/>
-            </geometry>
-        </visual>
-        <collision>
-            <origin xyz="0 0 0" rpy="0 0 0"/>
-            <geometry>
-                <mesh filename="package://agx_arm_urdf/piper_h/meshes/flange.stl"/>
-            </geometry>
-        </collision>
-    </link>
-    <joint name="flange_joint" type="fixed">
-        <origin xyz="0 0 0" rpy="0 0 0"/>
-        <parent link="link6"/>
-        <child link="flange_link"/>
-    </joint>
-    <link name="gripper_base">
-        <inertial>
-            <origin xyz="-0.000183807162235591 8.05033155577911E-05 0.0321436689908876" rpy="0 0 0"/>
-            <mass value="0.45"/>
-            <inertia ixx="0.00092934" ixy="0.00000034" ixz="-0.00000738" iyy="0.00071447" iyz="0.00000005" izz="0.00039442"/>
-        </inertial>
-        <visual>
-            <origin xyz="0 0 0" rpy="0 0 0"/>
-            <geometry>
-                <mesh filename="package://agx_arm_urdf/piper_h/meshes/dae/gripper_base.dae"/>
-            </geometry>
-        </visual>
-        <collision>
-            <origin xyz="0 0 0" rpy="0 0 0"/>
-            <geometry>
-                <mesh filename="package://agx_arm_urdf/piper_h/meshes/gripper_base.stl"/>
-            </geometry>
-        </collision>
-    </link>
-    <joint name="gripper_base_joint" type="fixed">
-        <origin xyz="0 0 0.0045" rpy="0 0 0"/>
-        <parent link="flange_link"/>
-        <child link="gripper_base"/>
-    </joint>
-    <link name="gripper_tcp"/>
-    <joint name="gripper_tcp_joint" type="fixed">
-        <origin xyz="0 0 0.138" rpy="0 0 0"/>
-        <parent link="gripper_base"/>
-        <child link="gripper_tcp"/>
-    </joint>
-    <link name="gripper_link"/>
-    <joint name="gripper" type="prismatic">
-        <origin xyz="0 0 0" rpy="0 0 0"/>
-        <parent link="gripper_base"/>
-        <child link="gripper_link"/>
-        <axis xyz="0 0 1"/>
-        <limit lower="0" upper="0.1" effort="10" velocity="3"/>
-    </joint>
-    <link name="gripper_link1">
-        <inertial>
-            <origin xyz="0.00065123185041968 -0.0491929869131989 0.00972258769184025" rpy="0 0 0"/>
-            <mass value="0.025"/>
-            <inertia ixx="0.00007371" ixy="-0.00000113" ixz="0.00000021" iyy="0.00000781" iyz="-0.00001372" izz="0.0000747"/>
-        </inertial>
-        <visual>
-            <origin xyz="0 0 0" rpy="0 0 0"/>
-            <geometry>
-                <mesh filename="package://agx_arm_urdf/piper_h/meshes/dae/gripper_link1.dae"/>
-            </geometry>
-        </visual>
-        <collision>
-            <origin xyz="0 0 0" rpy="0 0 0"/>
-            <geometry>
-                <mesh filename="package://agx_arm_urdf/piper_h/meshes/gripper_link1.stl"/>
-            </geometry>
-        </collision>
-    </link>
-    <joint name="gripper_joint1" type="prismatic">
-        <origin xyz="0 0 0.138" rpy="1.5707963 0 0"/>
-        <parent link="gripper_base"/>
-        <child link="gripper_link1"/>
-        <axis xyz="0 0 1"/>
-        <limit lower="0" upper="0.05" effort="10" velocity="3"/>
-        <mimic joint="gripper" multiplier="0.5" offset="0.0"/>
-    </joint>
-    <link name="gripper_link2">
-        <inertial>
-            <origin xyz="0.00065123185041968 -0.0491929869131989 0.00972258769184025" rpy="0 0 0"/>
-            <mass value="0.025"/>
-            <inertia ixx="0.00007371" ixy="-0.00000113" ixz="0.00000021" iyy="0.00000781" iyz="-0.00001372" izz="0.0000747"/>
-        </inertial>
-        <visual>
-            <origin xyz="0 0 0" rpy="0 0 0"/>
-            <geometry>
-                <mesh filename="package://agx_arm_urdf/piper_h/meshes/dae/gripper_link2.dae"/>
-            </geometry>
-        </visual>
-        <collision>
-            <origin xyz="0 0 0" rpy="0 0 0"/>
-            <geometry>
-                <mesh filename="package://agx_arm_urdf/piper_h/meshes/gripper_link2.stl"/>
-            </geometry>
-        </collision>
-    </link>
-    <joint name="gripper_joint2" type="prismatic">
-        <origin xyz="0 0 0.138" rpy="1.5707963 0 -3.1415926"/>
-        <parent link="gripper_base"/>
-        <child link="gripper_link2"/>
-        <axis xyz="0 0 -1"/>
-        <limit lower="-0.05" upper="0" effort="10" velocity="3"/>
-        <mimic joint="gripper" multiplier="-0.5" offset="0.0"/>
-    </joint>
+  <xacro:arg name="prefix" default=""/>
+  <xacro:include filename="$(find agx_arm_urdf)/piper_h/urdf/piper_h_with_gripper.xacro"/>
+  <xacro:piper_h_with_gripper prefix="$(arg prefix)"/>
+  <link name="world"/>
+  <joint name="world_to_$(arg prefix)base_link" type="fixed">
+    <parent link="world"/>
+    <child link="$(arg prefix)base_link"/>
+    <origin xyz="0 0 0" rpy="0 0 0"/>
+  </joint>
 </robot>
