Commit message: add inertia to gripper model

File: gripper/urdf/agx_gripper.xacro (robot description, xacro)
@@ -58,5 +58,12 @@
       <child link="${prefix}gripper_tcp"/>
     </joint>
-    <link name="${prefix}gripper_link"/>
+    <link name="${prefix}gripper_link">
+      <!-- Keep the virtual actuator link when Gazebo converts the URDF to SDF. -->
+      <inertial>
+        <origin xyz="0 0 0" rpy="0 0 0"/>
+        <mass value="0.001"/>
+        <inertia ixx="1e-6" ixy="0" ixz="0" iyy="1e-6" iyz="0" izz="1e-6"/>
+      </inertial>
+    </link>
     <joint name="${prefix}gripper" type="prismatic">
       <origin xyz="0 0 0" rpy="0 0 0"/>
