Commit message: update joint limits and max. velocities given the datasheet

File: piper_h/urdf/piper_h_arm.xacro (robot description, xacro)
@@ -1,3 +1,6 @@
 <?xml version="1.0"?>
+<!-- Joint position and velocity limits: PiPER X/H/L datasheet, page 3.
+     https://www.agilex-italia.it/wp-content/uploads/2025/08/PiPER-XHL-EN.pdf
+     URDF units: radians and radians/second. -->
 <robot xmlns:xacro="http://www.ros.org/wiki/xacro">
   <xacro:macro name="piper_h_arm" params="prefix">
@@ -45,5 +48,5 @@
             <child link="${prefix}link1"/>
             <axis xyz="0 0 1"/>
-            <limit lower="-2.6179938" upper="2.6179938" effort="100" velocity="5"/>
+            <limit lower="-2.6878070481" upper="2.6878070481" effort="100" velocity="3.1415926536"/>
         </joint>
         <link name="${prefix}link2">
@@ -71,5 +74,5 @@
             <child link="${prefix}link2"/>
             <axis xyz="0 0 1"/>
-            <limit lower="0" upper="3.1415926" effort="100" velocity="5"/>
+            <limit lower="0.0000000000" upper="3.4033920414" effort="100" velocity="3.4033920414"/>
         </joint>
         <link name="${prefix}link3">
@@ -97,5 +100,5 @@
             <child link="${prefix}link3"/>
             <axis xyz="0 0 1"/>
-            <limit lower="-2.9670597" upper="0" effort="100" velocity="5"/>
+            <limit lower="-3.0543261910" upper="0.0000000000" effort="100" velocity="3.1415926536"/>
         </joint>
         <link name="${prefix}link4">
@@ -123,5 +126,5 @@
             <child link="${prefix}link4"/>
             <axis xyz="0 0 1"/>
-            <limit lower="-2.3561944" upper="2.3561944" effort="100" velocity="5"/>
+            <limit lower="-2.2165681500" upper="2.2165681500" effort="100" velocity="3.9269908170"/>
         </joint>
         <link name="${prefix}link5">
@@ -149,5 +152,5 @@
             <child link="${prefix}link5"/>
             <axis xyz="0 0 1"/>
-            <limit lower="-1.5620696" upper="1.5620696" effort="100" velocity="5"/>
+            <limit lower="-1.5707963268" upper="1.5707963268" effort="100" velocity="3.9269908170"/>
         </joint>
         <link name="${prefix}link6">
@@ -175,5 +178,5 @@
             <child link="${prefix}link6"/>
             <axis xyz="0 0 1"/>
-            <limit lower="-2.0943951" upper="2.0943951" effort="100" velocity="5"/>
+            <limit lower="-2.9670597284" upper="2.9670597284" effort="100" velocity="3.9269908170"/>
         </joint>
   </xacro:macro>

File: piper_h/urdf/piper_h_description.urdf (robot description, URDF)
Before this commit: robot piper_h, 8 links, 7 joints
Joints:
- joint joint1: limit lower=-2.6179938 upper=2.6179938 effort=100 velocity=5 -> lower=-2.6878070481 upper=2.6878070481 effort=100 velocity=3.1415926536
- joint joint2: limit lower=0 upper=3.1415926 effort=100 velocity=5 -> lower=0.0000000000 upper=3.4033920414 effort=100 velocity=3.4033920414
- joint joint3: limit lower=-2.9670597 upper=0 effort=100 velocity=5 -> lower=-3.0543261910 upper=0.0000000000 effort=100 velocity=3.1415926536
- joint joint4: limit lower=-2.3561944 upper=2.3561944 effort=100 velocity=5 -> lower=-2.2165681500 upper=2.2165681500 effort=100 velocity=3.9269908170
- joint joint5: limit lower=-1.5620696 upper=1.5620696 effort=100 velocity=5 -> lower=-1.5707963268 upper=1.5707963268 effort=100 velocity=3.9269908170
- joint joint6: limit lower=-2.0943951 upper=2.0943951 effort=100 velocity=5 -> lower=-2.9670597284 upper=2.9670597284 effort=100 velocity=3.9269908170

File: piper_l/urdf/piper_l_arm.xacro (robot description, xacro)
@@ -1,3 +1,6 @@
 <?xml version="1.0"?>
+<!-- Joint position and velocity limits: PiPER X/H/L datasheet, page 3.
+     https://www.agilex-italia.it/wp-content/uploads/2025/08/PiPER-XHL-EN.pdf
+     URDF units: radians and radians/second. -->
 <robot xmlns:xacro="http://www.ros.org/wiki/xacro">
   <xacro:macro name="piper_l_arm" params="prefix">
@@ -45,5 +48,5 @@
             <child link="${prefix}link1"/>
             <axis xyz="0 0 1"/>
-            <limit lower="-2.6179938" upper="2.6179938" effort="100" velocity="5"/>
+            <limit lower="-2.6878070481" upper="2.6878070481" effort="100" velocity="3.1415926536"/>
         </joint>
         <link name="${prefix}link2">
@@ -71,5 +74,5 @@
             <child link="${prefix}link2"/>
             <axis xyz="0 0 1"/>
-            <limit lower="0" upper="3.1415926" effort="100" velocity="5"/>
+            <limit lower="0.0000000000" upper="3.4033920414" effort="100" velocity="3.4033920414"/>
         </joint>
         <link name="${prefix}link3">
@@ -97,5 +100,5 @@
             <child link="${prefix}link3"/>
             <axis xyz="0 0 1"/>
-            <limit lower="-2.9670597" upper="0" effort="100" velocity="5"/>
+            <limit lower="-3.0543261910" upper="0.0000000000" effort="100" velocity="3.1415926536"/>
         </joint>
         <link name="${prefix}link4">
@@ -123,5 +126,5 @@
             <child link="${prefix}link4"/>
             <axis xyz="0 0 1"/>
-            <limit lower="-2.2165681" upper="2.2165681" effort="100" velocity="5"/>
+            <limit lower="-2.2165681500" upper="2.2165681500" effort="100" velocity="3.9269908170"/>
         </joint>
         <link name="${prefix}link5">
@@ -149,5 +152,5 @@
             <child link="${prefix}link5"/>
             <axis xyz="0 0 1"/>
-            <limit lower="-1.5620696" upper="1.5620696" effort="100" velocity="5"/>
+            <limit lower="-1.5707963268" upper="1.5707963268" effort="100" velocity="3.9269908170"/>
         </joint>
         <link name="${prefix}link6">
@@ -175,5 +178,5 @@
             <child link="${prefix}link6"/>
             <axis xyz="0 0 1"/>
-            <limit lower="-2.0943951" upper="2.0943951" effort="100" velocity="5"/>
+            <limit lower="-2.9670597284" upper="2.9670597284" effort="100" velocity="3.9269908170"/>
         </joint>
   </xacro:macro>

File: piper_l/urdf/piper_l_description.urdf (robot description, URDF)
Before this commit: robot piper_l, 8 links, 7 joints
Joints:
- joint joint1: limit lower=-2.6179938 upper=2.6179938 effort=100 velocity=5 -> lower=-2.6878070481 upper=2.6878070481 effort=100 velocity=3.1415926536
- joint joint2: limit lower=0 upper=3.1415926 effort=100 velocity=5 -> lower=0.0000000000 upper=3.4033920414 effort=100 velocity=3.4033920414
- joint joint3: limit lower=-2.9670597 upper=0 effort=100 velocity=5 -> lower=-3.0543261910 upper=0.0000000000 effort=100 velocity=3.1415926536
- joint joint4: limit lower=-2.2165681 upper=2.2165681 effort=100 velocity=5 -> lower=-2.2165681500 upper=2.2165681500 effort=100 velocity=3.9269908170
- joint joint5: limit lower=-1.5620696 upper=1.5620696 effort=100 velocity=5 -> lower=-1.5707963268 upper=1.5707963268 effort=100 velocity=3.9269908170
- joint joint6: limit lower=-2.0943951 upper=2.0943951 effort=100 velocity=5 -> lower=-2.9670597284 upper=2.9670597284 effort=100 velocity=3.9269908170

File: piper_x/urdf/piper_x_arm.xacro (robot description, xacro)
@@ -1,3 +1,6 @@
 <?xml version="1.0"?>
+<!-- Joint position and velocity limits: PiPER X/H/L datasheet, page 3.
+     https://www.agilex-italia.it/wp-content/uploads/2025/08/PiPER-XHL-EN.pdf
+     URDF units: radians and radians/second. -->
 <robot xmlns:xacro="http://www.ros.org/wiki/xacro">
   <xacro:macro name="piper_x_arm" params="prefix">
@@ -45,5 +48,5 @@
             <child link="${prefix}link1"/>
             <axis xyz="0 0 1"/>
-            <limit lower="-2.6179938" upper="2.6179938" effort="100" velocity="5"/>
+            <limit lower="-2.6878070481" upper="2.6878070481" effort="100" velocity="3.1415926536"/>
         </joint>
         <link name="${prefix}link2">
@@ -71,5 +74,5 @@
             <child link="${prefix}link2"/>
             <axis xyz="0 0 1"/>
-            <limit lower="0" upper="3.1415926" effort="100" velocity="5"/>
+            <limit lower="0.0000000000" upper="3.4033920414" effort="100" velocity="3.4033920414"/>
         </joint>
         <link name="${prefix}link3">
@@ -97,5 +100,5 @@
             <child link="${prefix}link3"/>
             <axis xyz="0 0 1"/>
-            <limit lower="-2.9670597" upper="0" effort="100" velocity="5"/>
+            <limit lower="-3.0543261910" upper="0.0000000000" effort="100" velocity="3.1415926536"/>
         </joint>
         <link name="${prefix}link4">
@@ -123,5 +126,5 @@
             <child link="${prefix}link4"/>
             <axis xyz="0 0 1"/>
-            <limit lower="-1.553343" upper="1.553343" effort="100" velocity="5"/>
+            <limit lower="-1.5707963268" upper="1.5707963268" effort="100" velocity="3.9269908170"/>
         </joint>
         <link name="${prefix}link5">
@@ -149,5 +152,5 @@
             <child link="${prefix}link5"/>
             <axis xyz="0 0 1"/>
-            <limit lower="-1.553343" upper="1.553343" effort="100" velocity="5"/>
+            <limit lower="-1.5707963268" upper="1.5707963268" effort="100" velocity="3.9269908170"/>
         </joint>
         <link name="${prefix}link6">
@@ -175,5 +178,5 @@
             <child link="${prefix}link6"/>
             <axis xyz="0 0 1"/>
-            <limit lower="-2.0943951" upper="2.0943951" effort="100" velocity="5"/>
+            <limit lower="-2.8797932658" upper="2.8797932658" effort="100" velocity="3.9269908170"/>
         </joint>
   </xacro:macro>

File: piper_x/urdf/piper_x_description.urdf (robot description, URDF)
Before this commit: robot piper_x, 8 links, 7 joints
Joints:
- joint joint1: limit lower=-2.6179938 upper=2.6179938 effort=100 velocity=5 -> lower=-2.6878070481 upper=2.6878070481 effort=100 velocity=3.1415926536
- joint joint2: limit lower=0 upper=3.1415926 effort=100 velocity=5 -> lower=0.0000000000 upper=3.4033920414 effort=100 velocity=3.4033920414
- joint joint3: limit lower=-2.9670597 upper=0 effort=100 velocity=5 -> lower=-3.0543261910 upper=0.0000000000 effort=100 velocity=3.1415926536
- joint joint4: limit lower=-1.553343 upper=1.553343 effort=100 velocity=5 -> lower=-1.5707963268 upper=1.5707963268 effort=100 velocity=3.9269908170
- joint joint5: limit lower=-1.553343 upper=1.553343 effort=100 velocity=5 -> lower=-1.5707963268 upper=1.5707963268 effort=100 velocity=3.9269908170
- joint joint6: limit lower=-2.0943951 upper=2.0943951 effort=100 velocity=5 -> lower=-2.8797932658 upper=2.8797932658 effort=100 velocity=3.9269908170
